File: CE346 PCB/_autosave-CE346 PCB.kicad_sch (KiCad schematic)
At the start: 10 parts, among them IC1 nRF52833-QDAA-R, J1 Conn_01x04_Pin, J2 Conn_01x04_Pin, J3 Conn_02x04_Odd_Even, J4 Conn_02x04_Odd_Even, U1 ESP32-WROOM-32E-N4, Y1 Crystal_GND23

Commit message: schem
Parts:
- removed J1, J2: Conn_01x04_Pin, symbol Connector:Conn_01x04_Pin
- added D2: D_Zener, symbol Device:D_Zener
- added J1, J2: Conn_02x04_Odd_Even, symbol Connector_Generic:Conn_02x04_Odd_Even
- added MK1, MK2, MK3, MK4, MK5: IM69D130, CE346 Footprints:Logic_level_shifter, symbol Sensor_Audio:IM69D130
- added R1: R, symbol Device:R
Connections:
- net at D1.1 (K): now also R1.2
- net at D1.2 (A): now also D2.2 (A)
Other:
- note added: "1x4 connectors for IR muxs (signal, data, power, gnd, and gnd for shielding)"
- note added: "logic level shifters"
- note added: "zener based protection (both + and - spikes)"
- note removed: "1x4 connectors for IR muxs (signal, data, power, gnd)"
- moved on the sheet: D1

Commit message: better schematic
Parts:
- removed J2, J4: Conn_02x04_Odd_Even, symbol Connector_Generic:Conn_02x04_Odd_Even
- added C3, C4, C5, C6, C7, C8: C, symbol Device:C
- added D10, D3, D4, D5, D6, D7, D8, D9: D_Zener, symbol Device:D_Zener
- added J10, J5, J7, J8, J9: Conn_01x03_Pin, symbol Connector:Conn_01x03_Pin
- added J2: Conn_01x02_Pin, symbol Connector:Conn_01x02_Pin
- added J4, J6: micro usb, 629105150921:WURTH_629105150921, symbol CE346 Symbols:micro usb
- added R10, R11, R12, R9: 1M, symbol Device:R
- added R2, R3: R, symbol Device:R
- added R4, R5, R6, R7, R8: 330, symbol Device:R
- added SW1, SW2: SW_Push, symbol Switch:SW_Push
- added U2: SN74LV1T32DCKRG4, DCK0005A_N, symbol CE346 Symbols:SN74LV1T32DCKRG4
- J1, J3: footprint (none) -> CE346 Footprints:2x4 jst
- R1: value R -> 1M
Connections:
- net +5V: now reaches MK2.2 (VDD)
- net +5V: now also MK1.2 (VDD), MK3.2 (VDD), MK4.2 (VDD), MK5.2 (VDD)
- net +3.3V: now reaches J1.1 (Pin_1)
- net +3.3V: now also R2.2, R3.1
- net IR_MUX_CTRL: now reaches J1.2 (Pin_2)
- net IR_MUX_DATA: now reaches J1.3 (Pin_3)
- net GND: now reaches J1.4 (Pin_4)
- net GND: now also C1.2, C2.2, J1.5 (Pin_5), J1.6 (Pin_6), J1.7 (Pin_7), J1.8 (Pin_8), Y1.2, Y1.3, C3.2, C4.2, C5.2, C6.2, C7.2, C8.2, J10.1 (Pin_1), J10.3 (Pin_3), J5.1 (Pin_1), J5.3 (Pin_3), J7.1 (Pin_1), J7.3 (Pin_3), J8.1 (Pin_1), J8.3 (Pin_3), J9.1 (Pin_1), J9.3 (Pin_3), R2.1, R3.2, SW1.1, SW2.2
- net at U1.3 (EN): now also SW1.2
- net CLK1: now reaches Y1.1
- net CLK1: now also C2.1, IC1.28 (XC1)
- net CLK2: now reaches Y1.4
- net CLK2: now also C1.1, IC1.29 (XC2)
- net PIEZO_1+: now reaches J3.1 (Pin_1)
- net PIEZO_1-: now reaches J3.2 (Pin_2)
- net PIEZO_2+: now reaches J3.3 (Pin_3)
- net PIEZO_2-: now reaches J3.4 (Pin_4)
- net PIEZO_3+: now reaches J3.5 (Pin_5)
- net PIEZO_3-: now reaches J3.6 (Pin_6)
- net PIEZO_4+: now reaches J3.7 (Pin_7)
- net PIEZO_4-: now reaches J3.8 (Pin_8)
- net at IC1.1 (DEC1): now also C5.1
- net at IC1.11 (DECUSB): now also C8.1
- net at IC1.16 (P0.18/NRESET): now also SW2.1
- net at IC1.21 (DEC5): now also C7.1
- net at IC1.26 (DEC6): now also C4.1
- net at IC1.27 (DEC3): now also C3.1
- net at IC1.38 (DEC4): now also C6.1
- net SPI_SCK: now reaches IC1.4 (P0.04/AIN2)
- new net: J8.2 (Pin_2), R6.1
- new net: J5.2 (Pin_2), R4.1
- new net: J7.2 (Pin_2), R5.1
- new net: D7.1 (K), R11.2
- new net: D7.2 (A), D8.2 (A)
- new net: D3.1 (K), R9.2
- new net: J9.2 (Pin_2), R8.1
- new net: D10.2 (A), D9.2 (A)
- new net: D3.2 (A), D4.2 (A)
- new net: D5.1 (K), R10.2
- new net: D5.2 (A), D6.2 (A)
- new net: D9.1 (K), R12.2
- new net: J10.2 (Pin_2), R7.1
- new net LED1: R4.2
- new net LED2: R5.2
- new net LED3: R6.2
- new net LED4: R8.2
- new net LED5: R7.2
Other:
- note added: "2x4 connectors for IR muxs (signal, data, power, gnd, and gnd for shielding) 2x gnd for control, 2x gnd for input"
- note added: "5 data pins for LEDs"
- note added: "Microphone"
- note added: "micro usb to program esp32"
- note added: "micro usb to program nrf"
- note added: "uart between esps"
- note removed: "1x4 connectors for IR muxs (signal, data, power, gnd, and gnd for shielding)"
- moved on the sheet: C1, C2, D1, D2, IC1, J1, MK1, MK2, MK3, MK4, MK5, R1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
