File: CE346 PCB/CE346 PCB.kicad_sch (KiCad schematic)
At the start: 2 parts, among them IC1 nRF52833-QDAA-R, U1 ESP32-WROOM-32E-N4

Commit message: schem
Parts:
- added C1, C2, C3, C4, C5, C6, C7, C8: C, symbol Device:C
- added D1, D10, D2, D3, D4, D5, D6, D7, D8, D9: D_Zener, symbol Device:D_Zener
- added J1, J3: Conn_02x04_Odd_Even, CE346 Footprints:2x4 jst, symbol Connector_Generic:Conn_02x04_Odd_Even
- added J10, J5, J7, J8, J9: Conn_01x03_Pin, symbol Connector:Conn_01x03_Pin
- added J2: Conn_01x02_Pin, symbol Connector:Conn_01x02_Pin
- added J4, J6: micro usb, 629105150921:WURTH_629105150921, symbol CE346 Symbols:micro usb
- added MK1, MK2, MK3, MK4, MK5: IM69D130, CE346 Footprints:Logic_level_shifter, symbol Sensor_Audio:IM69D130
- added R1, R10, R11, R12, R9: 1M, symbol Device:R
- added R2, R3: R, symbol Device:R
- added R4, R5, R6, R7, R8: 330, symbol Device:R
- added SW1, SW2: SW_Push, symbol Switch:SW_Push
- added U2: SN74LV1T32DCKRG4, DCK0005A_N, symbol CE346 Symbols:SN74LV1T32DCKRG4
- added Y1: Crystal_GND23, symbol Device:Crystal_GND23
Connections:
- net ESP_CS: now reaches U1.29 (IO5)
- net at U1.3 (EN): now also SW1.2
- net SPI_SCK: now reaches U1.30 (IO18)
- net SPI_SCK: now also IC1.4 (P0.04/AIN2)
- net SPI_MOSI: now reaches U1.31 (IO19)
- net SPI_MOSI: now also IC1.31 (P0.03/AIN1)
- net SPI_MISO: now reaches U1.37 (IO23)
- net SPI_MISO: now also IC1.32 (P0.02/AIN0)
- net at IC1.1 (DEC1): now also C5.1
- net at IC1.11 (DECUSB): now also C8.1
- net at IC1.16 (P0.18/NRESET): now also SW2.1
- net at IC1.21 (DEC5): now also C7.1
- net at IC1.26 (DEC6): now also C4.1
- net at IC1.27 (DEC3): now also C3.1
- net CLK1: now reaches IC1.28 (XC1)
- net CLK1: now also C2.1, Y1.1
- net CLK2: now reaches IC1.29 (XC2)
- net CLK2: now also C1.1, Y1.4
- net at IC1.38 (DEC4): now also C6.1
- net NRF_CS: now reaches IC1.5 (P0.05/AIN3)
- new net: J8.2 (Pin_2), R6.1
- new net: J5.2 (Pin_2), R4.1
- new net: D1.1 (K), R1.2
- new net: J7.2 (Pin_2), R5.1
- new net: D7.1 (K), R11.2
- new net: D7.2 (A), D8.2 (A)
- new net: D1.2 (A), D2.2 (A)
- new net: D3.1 (K), R9.2
- new net: J9.2 (Pin_2), R8.1
- new net: D10.2 (A), D9.2 (A)
- new net: D3.2 (A), D4.2 (A)
- new net: D5.1 (K), R10.2
- new net: D5.2 (A), D6.2 (A)
- new net: D9.1 (K), R12.2
- new net: J10.2 (Pin_2), R7.1
- new net +3.3V: J1.1 (Pin_1), R2.2, R3.1
- new net +5V: MK1.2 (VDD), MK2.2 (VDD), MK3.2 (VDD), MK4.2 (VDD), MK5.2 (VDD)
- new net GND: C1.2, C2.2, C3.2, C4.2, C5.2, C6.2, C7.2, C8.2, J1.4 (Pin_4), J1.5 (Pin_5), J1.6 (Pin_6), J1.7 (Pin_7), J1.8 (Pin_8), J10.1 (Pin_1), J10.3 (Pin_3), J5.1 (Pin_1), J5.3 (Pin_3), J7.1 (Pin_1), J7.3 (Pin_3), J8.1 (Pin_1), J8.3 (Pin_3), J9.1 (Pin_1), J9.3 (Pin_3), R2.1, R3.2, SW1.1, SW2.2, Y1.2, Y1.3
- new net IR_MUX_CTRL: J1.2 (Pin_2)
- new net IR_MUX_DATA: J1.3 (Pin_3)
- new net LED1: R4.2
- new net LED2: R5.2
- new net LED3: R6.2
- new net LED4: R8.2
- new net LED5: R7.2
- new net PIEZO_1+: J3.1 (Pin_1)
- new net PIEZO_1-: J3.2 (Pin_2)
- new net PIEZO_2+: J3.3 (Pin_3)
- new net PIEZO_2-: J3.4 (Pin_4)
- new net PIEZO_3+: J3.5 (Pin_5)
- new net PIEZO_3-: J3.6 (Pin_6)
- new net PIEZO_4+: J3.7 (Pin_7)
- new net PIEZO_4-: J3.8 (Pin_8)
Other:
- note added: "2x4 connectors for 4 piezo sensors"
- note added: "2x4 connectors for IR muxs (signal, data, power, gnd, and gnd for shielding) 2x gnd for control, 2x gnd for input"
- note added: "32MHz clk"
- note added: "5 data pins for LEDs"
- note added: "Microphone"
- note added: "logic level shifters"
- note added: "micro usb to program esp32"
- note added: "micro usb to program nrf"
- note added: "uart between esps"
- note added: "zener based protection (both + and - spikes)"
- moved on the sheet: IC1, U1

Commit message: small changes
Parts:
- added R13, R14, R15, R16, R17: 330, symbol Device:R
Connections:
- net IR_MUX_CTRL is gone; now on net IR_MUX_CTRL1: J1.2 (Pin_2)
- net GND: no longer J1.4 (Pin_4), J1.6 (Pin_6)
- net IR_MUX_DATA: now also IC1.36 (P0.31/AIN7)
- net LED1: now also U1.6 (IO34)
- net LED2: now also U1.7 (IO35)
- net LED3: now also U1.8 (IO32)
- net LED4: now also U1.9 (IO33)
- net LED5: now also U1.10 (IO25)
- net at R1.1: now also D2.1 (K)
- net at D1.1 (K), R1.2: now also R13.1
- net at D7.1 (K), R11.2: now also R16.1
- net at R9.1: now also D4.1 (K)
- net at D3.1 (K), R9.2: now also R14.1
- net at D10.1 (K): now also R12.1
- net at D8.1 (K): now also R11.1
- net at D5.1 (K), R10.2: now also R15.1
- net at D6.1 (K): now also R10.1
- net at D9.1 (K), R12.2: now also R17.1
- net IR_MUX_CTRL1: now reaches IC1.14 (P0.15)
- net IR_MUX_CTRL2: now reaches IC1.15 (P0.17)
- net IR_MUX_CTRL2: now also J1.4 (Pin_4)
- net IR_MUX_CTRL3: now reaches IC1.17 (P0.20)
- net IR_MUX_CTRL3: now also J1.6 (Pin_6)
Other:
- moved on the sheet: R1, R10, R11, R12, R2, R9, SW2
