File: PCB/_autosave-CE346 PCB.kicad_sch (KiCad schematic)
At the start: 48 parts, among them IC1 nRF52833-QDAA-R, J1 Conn_02x04_Odd_Even, J10 Conn_01x03_Pin, J2 Conn_01x02_Pin, J3 Conn_02x04_Odd_Even, J5 Conn_01x03_Pin, J6 Conn_02x03_Counter_Clockwise, J7 Conn_01x03_Pin, J8 Conn_01x03_Pin, J9 Conn_01x03_Pin, SW2 SW_Push, U1 SN74LV1T32DCKRG4, U2 ESP32-WROOM-32E-N4, U3 SN74LV1T32DCKRG4, U4 SN74LV1T32DCKRG4, U5 SN74LV1T32DCKRG4, U6 SN74LV1T32DCKRG4, Y1 Crystal_GND23

Commit message: Updated comms code
Parts:
- removed D1, D2, D3, D4, D5, D6, D7, D8: D_Zener, symbol Device:D_Zener
- removed J10, J5, J7, J8, J9: Conn_01x03_Pin, symbol Connector:Conn_01x03_Pin
- removed J2: Conn_01x02_Pin, symbol Connector:Conn_01x02_Pin
- removed J6: Conn_02x03_Counter_Clockwise, symbol Connector_Generic:Conn_02x03_Counter_Clockwise
- removed R11: 1M, symbol Device:R
- removed U1, U3, U4: SN74LV1T32DCKRG4, DCK0005A_N, symbol CE346 Symbols:SN74LV1T32DCKRG4
- removed U2: ESP32-WROOM-32E-N4, symbol CE346 Symbols:ESP32-WROOM-32E-N4
- added C10, C11, C12, C29, C9: 0.1 uF, Capacitor_SMD:C_0402_1005Metric, symbol Device:C
- added C30: 4.7 uF, Capacitor_SMD:C_0805_2012Metric, symbol Device:C
- added D11, D12, D13, D14: 2.7 v Zenner, Diode_SMD:D_SOD-123, symbol Device:D_Zener
- added J10, J12, J2: Conn_01x02_Socket, Connector_PinHeader_2.54mm:PinHeader_1x02_P2.54mm_Vertical, symbol Connector:Conn_01x02_Socket
- added J11: Conn_01x06_Pin, Connector_PinHeader_2.54mm:PinHeader_1x06_P2.54mm_Vertical, symbol Connector:Conn_01x06_Pin
- added J14: Conn_01x05_Pin, Connector_PinHeader_2.54mm:PinHeader_1x05_P2.54mm_Vertical, symbol Connector:Conn_01x05_Pin
- added J15, J16, J17, J18: Conn_01x04_Pin, Connector_PinHeader_2.54mm:PinHeader_1x04_P2.54mm_Vertical, symbol Connector:Conn_01x04_Pin
- added J4, J5, J6, J7, J8, J9: Conn_01x02_Pin, Connector_PinHeader_2.54mm:PinHeader_1x02_P2.54mm_Vertical, symbol Connector:Conn_01x02_Pin
- added LED4: Blue, LED_SMD:LED_0603_1608Metric, symbol Device:LED
- added R19, R20, R21, R22: 330, Resistor_SMD:R_0805_2012Metric, symbol Device:R
- added R23: 10 k, Resistor_SMD:R_0805_2012Metric, symbol Device:R
- added R24: 330R, Capacitor_SMD:C_0402_1005Metric, symbol Device:R
- added R3: 10k, Resistor_SMD:R_0805_2012Metric, symbol Device:R
- added SW1, SW3: SW_Push, CE346 Footprints:pushbutton, symbol Switch:SW_Push
- added U2, U7, U8: SN74LV1T32DCKRG4, CE346 Footprints:DBV0005A_N, symbol CE346 Symbols:SN74LV1T32DCKRG4
- added U3: ESP32-WROOM-32E-N4, esp:ESP32­WROOM­32E_EXP, symbol CE346 Symbols:ESP32-WROOM-32E-N4
- added U4: MP34DT05TR-A, CE346 Footprints:MP34DT05TR-A_STM, symbol 2026-05-14_17-03-08:MP34DT05TR-A
- added U9: LDL1117S30R, CE346 Footprints:SOT223_STM, symbol 2026-04-27_01-58-37:LDL1117S30R
- C1, C2: value C -> 12 pF; footprint (none) -> Capacitor_SMD:C_0402_1005Metric
- C3: value C -> 100 pF; footprint (none) -> Capacitor_SMD:C_0402_1005Metric
- C4: value C -> 1.0 uF; footprint (none) -> Capacitor_SMD:C_0402_1005Metric
- C5: value C -> 100 nF; footprint (none) -> Capacitor_SMD:C_0402_1005Metric
- C6: value C -> 0.1 uF; footprint (none) -> Capacitor_SMD:C_0402_1005Metric
- C7: value C -> 820 pF; footprint (none) -> Capacitor_SMD:C_0402_1005Metric
- C8: value C -> 22 uF; footprint (none) -> Capacitor_SMD:C_0805_2012Metric
- IC1: footprint QFN40P500X500X90-41N -> nrf:QFN40_5X5_DQ_NOR-L
- R1: value 1M -> 10 k; footprint (none) -> Resistor_SMD:R_0805_2012Metric
- R10, R9: value 1M -> 10k; footprint (none) -> Resistor_SMD:R_0805_2012Metric
- R13, R14, R15, R16: value 330 -> 1M; footprint (none) -> Resistor_SMD:R_0805_2012Metric
- R2: value R -> 10k; footprint (none) -> Resistor_SMD:R_0805_2012Metric
- R4, R5, R6, R7, R8: footprint (none) -> Resistor_SMD:R_0805_2012Metric
- SW2: footprint (none) -> CE346 Footprints:pushbutton
- U5, U6: footprint DCK0005A_N -> CE346 Footprints:DBV0005A_N
- Y1: footprint (none) -> CE346 Footprints:32MHz Crystal
Connections:
- net PIEZO_4- is gone; now on net GND: J3.8 (Pin_8)
- net +3.3V: no longer R2.2
- net GND: now also IC1.25 (VSS_PA), IC1.37 (VSS_1), IC1.41 (VSS_2), J3.2 (Pin_2), J3.4 (Pin_4), J3.6 (Pin_6), R13.1, R14.1, R15.1, R16.1, SW2.1, U5.2 (B), U6.2 (B), C10.2, C11.2, C12.2, C29.1, C30.1, C9.2, D11.2 (A), D12.2 (A), D13.2 (A), D14.2 (A), J10.1 (Pin_1), J11.2 (Pin_2), J12.1 (Pin_1), J14.2 (Pin_2), J15.2 (Pin_2), J15.4 (Pin_4), J16.2 (Pin_2), J17.2 (Pin_2), J17.4 (Pin_4), J18.2 (Pin_2), J18.4 (Pin_4), J2.1 (Pin_1), J4.2 (Pin_2), J5.2 (Pin_2), J6.2 (Pin_2), J7.2 (Pin_2), J8.2 (Pin_2), J9.2 (Pin_2), LED4.1 (K), SW1.1, SW3.1, U2.2 (B), U2.3 (GND), U3.1 (GND), U3.15 (GND), U3.38 (GND), U3.39 (GND), U3.40 (GND), U3.41 (GND), U3.42 (GND), U3.43 (GND), U3.44 (GND), U3.45 (GND), U3.46 (GND), U3.47 (GND), U4.2 (LR), U4.5 (GND), U7.2 (B), U7.3 (GND), U8.2 (B), U8.3 (GND), U9.1 (GND); no longer J1.8 (Pin_8), R2.1, SW2.2
- net NRST: now also IC1.16 (P0.18/NRESET), R1.2, J14.5 (Pin_5), SW1.2
- net PIEZO_1+: now also R13.2, D11.1 (K), R19.1; no longer R1.2, R13.1
- net PIEZO_2+: now also R14.2, D12.1 (K), R20.1; no longer R14.1, R9.2
- net PIEZO_3+: now also R15.2, D13.1 (K), R21.1; no longer R10.2, R15.1
- net PIEZO_4+: now also R16.2, D14.1 (K), R22.1; no longer R16.1
- net SWDIO: now also IC1.19 (SWDIO), J14.3 (Pin_3)
- net at R6.1: now also J8.1 (Pin_1)
- net at R4.1: now also J4.1 (Pin_1)
- net at R5.1: now also J7.1 (Pin_1)
- net at R8.1: now also J5.1 (Pin_1)
- net DEC 4/6: now reaches C4.1, IC1.26 (DEC6)
- net DEC4/6: now reaches IC1.38 (DEC4)
- net DEC4/6: no longer C6.1
- net at IC1.11 (DECUSB): no longer C8.1
- net at R7.1: now also J6.1 (Pin_1)
- net VDD3V3: now reaches IC1.18 (VDD_2)
- net VDD3V3: now also C6.1, C8.1, IC1.30 (VDD_3), IC1.40 (VDD_4), IC1.8 (VDD_1), IC1.9 (VDDH), R1.1, R2.2, R9.2, C10.1, C11.1, C12.1, C30.2, C9.1, J11.1 (Pin_1), J14.1 (Pin_1), R23.1, R24.1, R3.2, U3.2 (3V3), U4.1 (VDD), U9.2 (VOUT), U9.4 (VOUT)
- net NRF_TX: now reaches IC1.2 (P0.00/XL1)
- net NRF_TX: now also J17.1 (Pin_1)
- net SWCLK: now reaches IC1.20 (SWDCLK)
- net SWCLK: now also J14.4 (Pin_4)
- net SCOREBOARD_RX: now reaches IC1.22 (P0.09/NFC1)
- net SCOREBOARD_RX: now also J15.3 (Pin_3)
- net SCOREBOARD_TX: now reaches IC1.23 (P0.10/NFC2)
- net SCOREBOARD_TX: now also J15.1 (Pin_1)
- net NRF_RX: now reaches IC1.3 (P0.01/XL2)
- net NRF_RX: now also J17.3 (Pin_3)
- net IR_MUX_CTRL_3: now reaches IC1.31 (P0.03/AIN1)
- net IR_MUX_CTRL_3: now also J1.2 (Pin_2)
- net SPI_SCK: now reaches IC1.4 (P0.04/AIN2)
- net SPI_SCK: now also U3.30 (IO18)
- net SPI_CS: now reaches IC1.5 (P0.05/AIN3)
- net SPI_CS: now also U3.29 (IO5)
- net SPI_MISO: now reaches IC1.6 (P1.09)
- net SPI_MISO: now also U3.37 (IO23)
- net SPI_MOSI: now reaches IC1.7 (P0.11)
- net SPI_MOSI: now also U3.31 (IO19)
- net +5V renamed VDD5V0
- net VDD5V0: now also C29.2, J16.1 (Pin_1), J9.1 (Pin_1), U2.5 (VCC), U7.5 (VCC), U8.5 (VCC), U9.3 (VIN)
- net IR_MUX_CTRL1 renamed IR_MUX_CTRL_0
- net IR_MUX_CTRL_0: now also J1.8 (Pin_8); no longer J1.2 (Pin_2)
- net IR_MUX_CTRL2 renamed IR_MUX_CTRL_1
- net IR_MUX_CTRL_1: now also J1.6 (Pin_6); no longer J1.4 (Pin_4)
- net IR_MUX_CTRL3 renamed IR_MUX_CTRL_2
- net IR_MUX_CTRL_2: now also J1.4 (Pin_4); no longer J1.6 (Pin_6)
- net LED_IN4 renamed DIN3
- net DIN3: now also U3.8 (IO32)
- net LED_IN5 renamed DIN2
- net DIN2: now also U3.26 (IO4)
- net LED_OUT1 renamed LED1
- net LED1: now also U2.4 (Y)
- net LED_OUT2 renamed LED2
- net LED2: now also U5.4 (Y)
- net LED_OUT3 renamed LED3
- net LED3: now also U6.4 (Y)
- net LED_OUT4 renamed LED4
- net LED4: now also U7.4 (Y); no longer U6.4 (Y)
- net LED_OUT5 renamed LED5
- net LED5: now also U8.4 (Y); no longer U5.4 (Y)
- removed net PIEZO_1-: J3.2 (Pin_2), R1.1
- net PIEZO_1_OUT renamed PIEZO1
- net PIEZO1: now also R19.2; no longer R13.2
- net PIEZO_2- renamed sound_reactive_button
- net sound_reactive_button: now also J10.2 (Pin_2), U3.5 (SENSOR_VN); no longer J3.4 (Pin_4)
- net PIEZO_2_OUT renamed PIEZO2
- net PIEZO2: now also R20.2; no longer R14.2
- net PIEZO_3- renamed KILL_SWITCH
- net KILL_SWITCH: now also J12.2 (Pin_2), U3.4 (SENSOR_VP); no longer J3.6 (Pin_6)
- net PIEZO_3_OUT renamed PIEZO3
- net PIEZO3: now also R21.2; no longer R15.2
- net PIEZO_4_OUT renamed PIEZO4
- net PIEZO4: now also R22.2; no longer R16.2
- new net: R2.1, SW3.2, U3.25 (IO0)
- new net: R23.2, SW2.2, U3.3 (EN)
- new net: LED4.2 (A), R24.2
- new net BCLK: J11.3 (Pin_3), U3.13 (IO14)
- new net DIN1: U2.1 (A), U3.27 (IO16)
- new net DIN4: U3.9 (IO33), U7.1 (A)
- new net DIN5: U3.10 (IO25), U8.1 (A)
- new net DOUT: J11.5 (Pin_5), U3.36 (IO22)
- new net LRCL: J11.4 (Pin_4), U3.16 (IO13)
- new net PDM_CLK: U3.12 (IO27), U4.3 (CLK)
- new net PDM_DATA: U3.11 (IO26), U4.4 (DOUT)
- new net RX0: J16.4 (Pin_4), U3.34 (RXD0)
- new net SEL: J11.6 (Pin_6), U3.28 (IO17)
- new net TX0: J16.3 (Pin_3), U3.35 (TXD0)
- new net UART2_RX: J18.3 (Pin_3), U3.6 (IO34)
- new net UART2_TX: J18.1 (Pin_1), U3.33 (IO21)
- new net game_state_button: J2.2 (Pin_2), R3.1, U3.7 (IO35)
- no-connect marks 0 -> 9
Other:
- note removed: "Programming Header"
- moved on the sheet: C1, C2, C5, C7, IC1, R5, R6, R7, Y1
